Commit message: Prepare navigation branch without oversized terrain asset

File: Mars-rover/rover_description/urdf/aries_base.xacro (robot description, xacro)
@@ -35,5 +35,5 @@
         <parent link="base_link"/>
         <child link="imu_frame"/>
-        <origin xyz="0.0 0.0 0.08" rpy="0.0 0.0 0.0"/>
+        <origin xyz="0.2 0.0 0.2125" rpy="0.0 0.0 0.0"/>
     </joint>
     <!-- Base Footprint -->

File: Mars-rover/rover_description/urdf/aries_gazebo.xacro (robot description, xacro)
@@ -134,18 +134,7 @@
   <gazebo reference="Lidar_Link">
   </gazebo>
-  <!-- Gazebo Plugin for Joint State Publisher -->
-  <!-- When ros2_control is active (use_sim=true), only publish passive joints not managed by
-       joint_state_broadcaster. Wheel and aux joints are published by ros2_control instead. -->
-  <xacro:if value="$(arg use_sim)">
-    <gazebo>
-      <plugin filename="gz-sim-joint-state-publisher-system" name="gz::sim::systems::JointStatePublisher">
-        <topic>/joint_states</topic>
-        <joint_name>L_Rocker_Joint</joint_name>
-        <joint_name>R_Rocker_Joint</joint_name>
-        <joint_name>L_Boggie_Joint</joint_name>
-        <joint_name>R_Boggie_Joint</joint_name>
-      </plugin>
-    </gazebo>
-  </xacro:if>
+  <!-- Gazebo Plugin for Joint State Publisher (Only needed if ros2_control is not used) -->
+  <!-- When ros2_control is active (use_sim=true), gz_ros2_control's joint_state_broadcaster
+       publishes ALL joint states (wheels, suspension, rockers) in a single synchronized message. -->
   <xacro:unless value="$(arg use_sim)">
     <gazebo>
@@ -292,17 +281,4 @@
           <visualize>true</visualize>
           <topic>/imu</topic>
-          <!-- Without this, gz-sim's IMU zeroes yaw relative to whatever
-               orientation the model had when the sensor was instantiated
-               (spawn-relative), not true world orientation: roll/pitch
-               stay gravity-referenced (correct) but yaw silently drifts off
-               by however much the spawn pose was rotated (spawn_yaw in
-               my_robot.launch.py), which fed a wrong heading into the EKF
-               and desynced RViz's displayed orientation from Gazebo's real
-               one. Forcing world-fixed ENU makes yaw absolute. -->
-          <imu>
-              <orientation_reference_frame>
-                  <localization>ENU</localization>
-              </orientation_reference_frame>
-          </imu>
       </sensor>
   </gazebo>
@@ -317,10 +293,5 @@
         <right_joint>R_2_Wheel_Joint</right_joint>
         <right_joint>R_3_Wheel_Joint</right_joint>
-        <!-- True geometric track width from URDF forward kinematics (see
-             rover_controllers/config/diff_controller.yaml), was 0.45 which
-             didn't match the actual robot geometry. This plugin is inactive
-             under the default launch (use_sim:=true uses ros2_control
-             instead), but kept correct in case it's ever re-enabled. -->
-        <wheel_separation>0.7095</wheel_separation>
+        <wheel_separation>0.45</wheel_separation>
         <wheel_radius>0.1100</wheel_radius>
         <frame_id>odom</frame_id>

File: Mars-rover/rover_description/urdf/common_properties.xacro (robot description, xacro)
@@ -23,5 +23,5 @@
     <xacro:property name="enable_lidar" value="false"/>
     <!-- Enable D435i -->
-    <xacro:property name="enable_D435i" value="false"/>
+    <xacro:property name="enable_D435i" value="true"/>
     <!-- Enable ZED 2i -->
     <xacro:property name="enable_zed2i" value="true"/>

File: Mars-rover/rover_description/urdf/d435i.xacro (robot description, xacro)
@@ -24,5 +24,5 @@
     <!-- Camera body, with origin at bottom screw mount -->
     <joint name="camera_joint" type="fixed">
-        <origin xyz="0.2756 0.0025 0.2535" rpy="0 0 0"/>
+        <origin xyz="0.245 0 0.225" rpy="0 0 0"/>
         <parent link="base_link"/>
         <child link="camera_bottom_screw_frame"/>
@@ -164,5 +164,5 @@
                 <visualize>false</visualize>
                 <topic>camera/color/image_raw</topic>
-                <gz_frame_id>camera_color_optical_frame</gz_frame_id>
+                <gz_frame_id>camera_color_frame</gz_frame_id>
             </sensor>
             <!-- The infra1/infra2 render sensors were removed from simulation:
@@ -181,10 +181,10 @@
                     <clip>
                         <near>0.1</near>
-                        <far>100</far>
+                        <far>3.5</far>
                     </clip>
                     <noise>
                         <type>gaussian</type>
                         <mean>0.0</mean>
-                        <stddev>0.100</stddev>
+                        <stddev>0.005</stddev>
                     </noise>
                 </camera>
@@ -193,5 +193,5 @@
                 <visualize>false</visualize>
                 <topic>camera/depth/image_rect_raw</topic>
-                <gz_frame_id>camera_depth_optical_frame</gz_frame_id>
+                <gz_frame_id>camera_depth_frame</gz_frame_id>
             </sensor>
             <!-- IMU Sensor -->
@@ -254,5 +254,5 @@
                 </imu>
                 <topic>camera/imu/data</topic>
-                <gz_frame_id>camera_gyro_optical_frame</gz_frame_id>
+                <gz_frame_id>camera_gyro_frame</gz_frame_id>
             </sensor>
         </gazebo>

File: Mars-rover/rover_description/urdf/differential_link.xacro (robot description, xacro)
@@ -59,5 +59,5 @@
             <origin xyz="0 0 0" rpy="0 0 0" />
             <geometry>
-                <mesh filename="${mesh_location}/L_Rod_link.stl" />
+                <mesh filename="${mesh_location}/R_Rod_link.stl" />
             </geometry>
             <material name="">
@@ -68,5 +68,5 @@
             <origin xyz="0 0 0" rpy="0 0 0" />
             <geometry>
-                <mesh filename="${mesh_location}/L_Rod_link.stl" />
+                <mesh filename="${mesh_location}/R_Rod_link.stl" />
             </geometry>
         </collision>
@@ -159,5 +159,5 @@
             <origin xyz="0 0 0" rpy="0 0 0" />
             <geometry>
-                <mesh filename="${mesh_location}/R_Rod_link.stl" />
+                <mesh filename="${mesh_location}/L_Rod_link.stl" />
             </geometry>
             <material name="">
@@ -168,5 +168,5 @@
             <origin xyz="0 0 0" rpy="0 0 0" />
             <geometry>
-                <mesh filename="${mesh_location}/R_Rod_link.stl" />
+                <mesh filename="${mesh_location}/L_Rod_link.stl" />
             </geometry>
         </collision>

File: Mars-rover/rover_description/urdf/left_link.xacro (robot description, xacro)
@@ -17,12 +17,16 @@
             <origin xyz="0 0 0" rpy="0 0 0"/>
             <geometry>
-                <mesh filename="${mesh_location}/L_Rocker_Link.STL"/>
+                <mesh filename="${mesh_location}/left_rocker.stl"/>
             </geometry>
             <material name="silver"/>
         </visual>
         <collision>
-            <origin xyz="0 0 0" rpy="0 0 0"/>
+            <!-- Box proxy, not the hi-poly visual mesh: a 34k-triangle concave
+                 mesh as direct collision geometry destabilizes the physics
+                 solver on this closed rocker-bogie-differential loop
+                 (observed as a wheel getting yanked on ground contact). -->
+            <origin xyz="-0.0021 0.0625 0.0242" rpy="0 0 0"/>
             <geometry>
-                <mesh filename="${mesh_location}/L_Rocker_Link.STL"/>
+                <box size="0.5044 0.2750 0.0825"/>
             </geometry>
         </collision>
@@ -30,5 +34,5 @@
     <!-- Left Rocker Joint -->
     <joint name="L_Rocker_Joint" type="revolute">
-        <origin xyz="0 0.271 0.070999999999999" rpy="${-PI/2} 0 ${PI}"/>
+        <origin xyz="0 0.2842 0.070999999999999" rpy="${-PI/2} 0 ${PI}"/>
         <parent link="base_link"/>
         <child link="L_Rocker_Link"/>
@@ -37,8 +41,8 @@
         <dynamics damping="50" friction="50"/>
     </joint>
-    <!-- Left Wheel 3 -->
-    <link name="L_3_Wheel_Link">
+    <!-- Left Wheel 1 -->
+    <link name="L_1_Wheel_Link">
         <inertial>
-            <origin xyz="0 -0.0350608778434713 0" rpy="1.57 0 0"/>
+            <origin xyz="0 -0.0350608778434713 0" rpy="${-PI/2} 0 ${PI}"/>
             <mass value="${wheel_mass}"/>
             <inertia
@@ -51,12 +55,12 @@
         </inertial>
         <visual>
-            <origin xyz="0 0 0" rpy="1.57 0 0"/>
+            <origin xyz="0 0 0" rpy="${-PI/2} 0 ${PI}"/>
             <geometry>
-                <mesh filename="${mesh_location}/L_3_Wheel_Link.STL"/>
+                <mesh filename="${mesh_location}/L_1_Wheel_Link.STL"/>
             </geometry>
             <material name="blue"/>
         </visual>
         <collision>
-            <origin xyz="0 -0.035 0" rpy="1.57 0 0"/>
+            <origin xyz="0 -0.035 0" rpy="${PI/2} 0 0"/>
             <geometry>
                 <cylinder radius="${wheel_radius}" length="${wheel_thickness}"/>
@@ -64,9 +68,8 @@
         </collision>
     </link>
-    <!-- Left Wheel 3 Joint -->
-    <joint name="L_3_Wheel_Joint" type="continuous">
-        <origin xyz="0.14142135623731 0.141421356237309 -0.08667" rpy="1.57 -3.14 0"/>
+    <joint name="L_1_Wheel_Joint" type="continuous">
+        <origin xyz="0.12754 0.1674 -0.0953" rpy="${-PI/2} 0 ${PI}"/>
         <parent link="L_Boggie_Link"/>
-        <child link="L_3_Wheel_Link"/>
+        <child link="L_1_Wheel_Link"/>
         <axis xyz="0 1 0"/>
         <dynamics damping="0.01" friction="0.01"/>
@@ -75,5 +78,5 @@
     <link name="L_2_Wheel_Link">
         <inertial>
-            <origin xyz="0 -0.0350608778434713 0" rpy="1.57 0 0"/>
+            <origin xyz="0 -0.0350608778434713 0" rpy="${-PI/2} 0 ${PI}"/>
             <mass value="${wheel_mass}"/>
             <inertia
@@ -86,5 +89,5 @@
         </inertial>
         <visual>
-            <origin xyz="0 0 0" rpy="1.57 0 0"/>
+            <origin xyz="0 0 0" rpy="${-PI/2} 0 ${PI}"/>
             <geometry>
                 <mesh filename="${mesh_location}/L_2_Wheel_Link.STL"/>
@@ -93,5 +96,5 @@
         </visual>
         <collision>
-            <origin xyz="0 -0.035 0" rpy="1.57 0 0"/>
+            <origin xyz="0 -0.035 0" rpy="${PI/2} 0 0"/>
             <geometry>
                 <cylinder radius="${wheel_radius}" length="${wheel_thickness}"/>
@@ -99,7 +102,6 @@
         </collision>
     </link>
-    <!-- Left Wheel 2 Joint -->
     <joint name="L_2_Wheel_Joint" type="continuous">
-        <origin xyz="-0.141421356237308 0.141421356237311 -0.08667" rpy="1.57 -3.14 0"/>
+        <origin xyz="-0.12754 0.1674 -0.0953" rpy="${-PI/2} 0 ${PI}"/>
         <parent link="L_Boggie_Link"/>
         <child link="L_2_Wheel_Link"/>
@@ -107,8 +109,8 @@
         <dynamics damping="0.01" friction="0.01"/>
     </joint>
-    <!-- Left Wheel 1 -->
-    <link name="L_1_Wheel_Link">
+    <!-- Left Wheel 3 -->
+    <link name="L_3_Wheel_Link">
         <inertial>
-            <origin xyz="0 -0.0350608778434703 0" rpy="1.57 0 0"/>
+            <origin xyz="0 -0.0350608778434713 0" rpy="${-PI/2} 0 ${PI}"/>
             <mass value="${wheel_mass}"/>
             <inertia
@@ -121,12 +123,12 @@
         </inertial>
         <visual>
-            <origin xyz="0 0 0" rpy="1.57 0 0"/>
+            <origin xyz="0 0 0" rpy="${-PI/2} 0 ${PI}"/>
             <geometry>
-                <mesh filename="${mesh_location}/L_1_Wheel_Link.STL"/>
+                <mesh filename="${mesh_location}/L_3_Wheel_Link.STL"/>
             </geometry>
             <material name="blue"/>
         </visual>
         <collision>
-            <origin xyz="0 -0.035 0" rpy="1.57 0 0"/>
+            <origin xyz="0 -0.035 0" rpy="${PI/2} 0 0"/>
             <geometry>
                 <cylinder radius="${wheel_radius}" length="${wheel_thickness}"/>
@@ -134,9 +136,9 @@
         </collision>
     </link>
-    <!-- Left Wheel 1 Joint -->
-    <joint name="L_1_Wheel_Joint" type="continuous">
-        <origin xyz="-0.261 0.1785 -0.0759999999999989" rpy="1.57 -3.14 0"/>
+    <!-- Left Wheel 3 Joint -->
+    <joint name="L_3_Wheel_Joint" type="continuous">
+        <origin xyz="-0.2299 0.1602 -0.0953" rpy="${-PI/2} 0 ${PI}"/>
         <parent link="L_Rocker_Link"/>
-        <child link="L_1_Wheel_Link"/>
+        <child link="L_3_Wheel_Link"/>
         <axis xyz="0 1 0"/>
         <dynamics damping="0.01" friction="0.01"/>
@@ -158,12 +160,13 @@
             <origin xyz="0 0 0" rpy="0 0 0"/>
             <geometry>
-                <mesh filename="${mesh_location}/L_Boggie_Link.STL"/>
+                <mesh filename="${mesh_location}/left_bogie.stl"/>
             </geometry>
             <material name="silver"/>
         </visual>
         <collision>
-            <origin xyz="0 0 0" rpy="0 0 0"/>
+            <!-- Box proxy, not the hi-poly visual mesh; see rocker collision comment above. -->
+            <origin xyz="-0.0002 0.0949 0.0006" rpy="0 0 0"/>
             <geometry>
-                <mesh filename="${mesh_location}/L_Boggie_Link.STL"/>
+                <box size="0.3401 0.2299 0.0480"/>
             </geometry>
         </collision>
@@ -171,5 +174,5 @@
     <!-- Left Boggie Joint -->
     <joint name="L_Boggie_Joint" type="revolute">
-        <origin xyz="0.1401 -0.01938 0" rpy="0 0 0"/>
+        <origin xyz="0.195 0 0" rpy="0 0 0"/>
         <parent link="L_Rocker_Link"/>
         <child link="L_Boggie_Link"/>

File: Mars-rover/rover_description/urdf/my_robot.urdf.xacro (robot description, xacro)
@@ -12,4 +12,5 @@
     <xacro:include filename="left_link.xacro" />
     <xacro:include filename="right_link.xacro" />
+    <xacro:include filename="d435i.xacro" />
     <xacro:include filename="rover_control.xacro" />
     <!-- zed2i.xacro requires the zed_description package, which isn't

File: Mars-rover/rover_description/urdf/right_link.xacro (robot description, xacro)
@@ -17,12 +17,16 @@
             <origin xyz="0 0 0" rpy="0 0 0"/>
             <geometry>
-                <mesh filename="${mesh_location}/R_Rocker_Link.STL"/>
+                <mesh filename="${mesh_location}/right_rocker.stl"/>
             </geometry>
             <material name="silver"/>
         </visual>
         <collision>
-            <origin xyz="0 0 0" rpy="0 0 0"/>
-            <geometry>
-                <mesh filename="${mesh_location}/R_Rocker_Link.STL"/>
+            <!-- Box proxy, not the hi-poly visual mesh: a 34k-triangle concave
+                 mesh as direct collision geometry destabilizes the physics
+                 solver on this closed rocker-bogie-differential loop
+                 (observed as a wheel getting yanked on ground contact). -->
+            <origin xyz="-0.0022 -0.0625 0.0224" rpy="0 0 0"/>
+            <geometry>
+                <box size="0.5044 0.2750 0.0790"/>
             </geometry>
         </collision>
@@ -30,5 +34,5 @@
     <!-- Right Rocker Joint -->
     <joint name="R_Rocker_Joint" type="revolute">
-        <origin xyz="0 -0.271 0.070999999999999" rpy="${PI/2} 0 ${PI}"/>
+        <origin xyz="0 -0.2842 0.070999999999999" rpy="${PI/2} 0 ${PI}"/>
         <parent link="base_link"/>
         <child link="R_Rocker_Link"/>
@@ -40,8 +44,8 @@
         <dynamics damping="50" friction="50"/>
     </joint>
-    <!-- Right Wheel 3 -->
-    <link name="R_3_Wheel_Link">
-        <inertial>
-            <origin xyz="0 0.0350608778434713 0" rpy="-1.57 0 0"/>
+    <!-- Right Wheel 1 -->
+    <link name="R_1_Wheel_Link">
+        <inertial>
+            <origin xyz="0 0.0350608778434713 0" rpy="${PI/2} 0 ${PI}"/>
             <mass value="${wheel_mass}"/>
             <inertia
@@ -54,12 +58,12 @@
             </inertial>
         <visual>
-            <origin xyz="0 0 0" rpy="-1.57 0 0"/>
-            <geometry>
-                <mesh filename="${mesh_location}/R_3_Wheel_Link.STL"/>
+            <origin xyz="0 0 0" rpy="${PI/2} 0 ${PI}"/>
+            <geometry>
+                <mesh filename="${mesh_location}/R_1_Wheel_Link.STL"/>
             </geometry>
             <material name="blue"/>
         </visual>
         <collision>
-            <origin xyz="0 0.035 0" rpy="-1.57 0 0"/>
+            <origin xyz="0 0.035 0" rpy="${PI/2} 0 0"/>
             <geometry>
                 <cylinder radius="${wheel_radius}" length="${wheel_thickness}"/>
@@ -67,9 +71,8 @@
         </collision>
     </link>
-    <!-- Right Wheel 3 Joint -->
-    <joint name="R_3_Wheel_Joint" type="continuous">
-        <origin xyz="0.1542 -0.1266 -0.086" rpy=" 1.57 0 -3.14"/>
+    <joint name="R_1_Wheel_Joint" type="continuous">
+        <origin xyz="0.12754 -0.1674 -0.0953" rpy="${PI/2} 0 ${PI}"/>
         <parent link="R_Boggie_Link"/>
-        <child link="R_3_Wheel_Link"/>
+        <child link="R_1_Wheel_Link"/>
         <axis xyz="0 1 0"/>
         <dynamics damping="0.01" friction="0.01"/>
@@ -78,5 +81,5 @@
     <link name="R_2_Wheel_Link">
         <inertial>
-            <origin xyz="0 0.0350608778434713 0" rpy="-1.57 0 0"/>
+            <origin xyz="0 0.0350608778434713 0" rpy="${PI/2} 0 ${PI}"/>
             <mass value="${wheel_mass}"/>
             <inertia
@@ -89,5 +92,5 @@
         </inertial>
         <visual>
-            <origin xyz="0 0 0" rpy="-1.57 0 0"/>
+            <origin xyz="0 0 0" rpy="${PI/2} 0 ${PI}"/>
             <geometry>
                 <mesh filename="${mesh_location}/R_2_Wheel_Link.STL"/>
@@ -96,5 +99,5 @@
         </visual>
         <collision>
-            <origin xyz="0 0.035 0" rpy="-1.57 0 0"/>
+            <origin xyz="0 0.035 0" rpy="${PI/2} 0 0"/>
             <geometry>
                 <cylinder radius="${wheel_radius}" length="${wheel_thickness}"/>
@@ -104,5 +107,5 @@
     <!-- Right Wheel 2 Joint -->
     <joint name="R_2_Wheel_Joint" type="continuous">
-        <origin xyz="-0.1267 -0.1545 -0.086" rpy=" 1.57 0 -3.14"/>
+        <origin xyz="-0.12754 -0.1674 -0.0953" rpy="${PI/2} 0 ${PI}"/>
         <parent link="R_Boggie_Link"/>
         <child link="R_2_Wheel_Link"/>
@@ -110,8 +113,8 @@
         <dynamics damping="0.01" friction="0.01"/>
     </joint>
-    <!-- Right Wheel 1 -->
-    <link name="R_1_Wheel_Link">
-        <inertial>
-            <origin xyz="0 0.0350608778434713 0" rpy="-1.57 0 0"/>
+    <!-- Right Wheel 3 -->
+    <link name="R_3_Wheel_Link">
+        <inertial>
+            <origin xyz="0 0.0350608778434713 0" rpy="${PI/2} 0 ${PI}"/>
             <mass value="${wheel_mass}"/>
             <inertia
@@ -124,12 +127,12 @@
         </inertial>
         <visual>
-            <origin xyz="0 0 0" rpy="-1.57 0 0"/>
-            <geometry>
-                <mesh filename="${mesh_location}/R_1_Wheel_Link.STL"/>
+            <origin xyz="0 0 0" rpy="${PI/2} 0 ${PI}"/>
+            <geometry>
+                <mesh filename="${mesh_location}/R_3_Wheel_Link.STL"/>
             </geometry>
             <material name="blue"/>
         </visual>
         <collision>
-            <origin xyz="0 0.035 0" rpy="-1.57 0 0"/>
+            <origin xyz="0 0.035 0" rpy="${PI/2} 0 0"/>
             <geometry>
                 <cylinder radius="${wheel_radius}" length="${wheel_thickness}"/>
@@ -138,8 +141,8 @@
     </link>
     <!-- Right Wheel 3 Joint -->
-    <joint name="R_1_Wheel_Joint" type="continuous">
-        <origin xyz="-0.276 -0.1541 -0.0760000000000001" rpy=" 1.57 0 -3.14"/>
+    <joint name="R_3_Wheel_Joint" type="continuous">
+        <origin xyz="-0.2299 -0.1602 -0.0953" rpy="${PI/2} 0 ${PI}"/>
         <parent link="R_Rocker_Link"/>
-        <child link="R_1_Wheel_Link"/>
+        <child link="R_3_Wheel_Link"/>
         <axis xyz="0 1 0"/>
         <dynamics damping="0.01" friction="0.01"/>
@@ -161,12 +164,13 @@
             <origin xyz="0 0 0" rpy="0 0 0"/>
             <geometry>
-                <mesh filename="${mesh_location}/R_Boggie_Link.STL"/>
+                <mesh filename="${mesh_location}/right_bogie.stl"/>
             </geometry>
             <material name="silver"/>
         </visual>
         <collision>
-            <origin xyz="0 0 0" rpy="0 0 0"/>
-            <geometry>
-                <mesh filename="${mesh_location}/R_Boggie_Link.STL"/>
+            <!-- Box proxy, not the hi-poly visual mesh; see rocker collision comment above. -->
+            <origin xyz="0.0002 -0.0949 0.0006" rpy="0 0 0"/>
+            <geometry>
+                <box size="0.3401 0.2299 0.0480"/>
             </geometry>
         </collision>
@@ -174,5 +178,5 @@
     <!-- Right Boggie Joint -->
     <joint name="R_Boggie_Joint" type="revolute">
-        <origin xyz="0.1411 0.006899 0" rpy="0 0 0"/>
+        <origin xyz="0.195 0 0" rpy="0 0 0"/>
         <parent link="R_Rocker_Link"/>
         <child link="R_Boggie_Link"/>

File: Mars-rover/rover_description/urdf/rover_control.xacro (robot description, xacro)
@@ -10,4 +10,21 @@
         <plugin>gz_ros2_control/GazeboSimSystem</plugin>
       </hardware>
+      <!-- PASSIVE SUSPENSION JOINTS (read-only state interfaces for unified joint_states) -->
+      <joint name="L_Rocker_Joint">
+        <state_interface name="position"/>
+        <state_interface name="velocity"/>
+      </joint>
+      <joint name="R_Rocker_Joint">
+        <state_interface name="position"/>
+        <state_interface name="velocity"/>
+      </joint>
+      <joint name="L_Boggie_Joint">
+        <state_interface name="position"/>
+        <state_interface name="velocity"/>
+      </joint>
+      <joint name="R_Boggie_Joint">
+        <state_interface name="position"/>
+        <state_interface name="velocity"/>
+      </joint>
       <!-- ROCKER JOINTS -->
       <joint name="aux_L_Rocker_joint">
